File: hardware/pcb/kicad/lumi/lumi.kicad_pcb (KiCad board)
At the start: 2 copper layers, 31 x 33 mm, 44 parts, among them J1 USB-C 16P, J2 FH12-30S-0.5SH, SW1 MSK12C02, U1 ESP32-C3-WROOM-02-N4, U2 LIS2DH12TR, U3 TP4054, U4 RT9080-33GJ5

Commit message: Lumi PCB: rebuild in KiCad 10 with datasheet fixes
Checking the draft against the panel and Espressif datasheets found faults
the design-rule check can't see: a mirrored panel at J2, a bottom-contact
connector where the panel needs top contact, a screen cable that couldn't
reach, VBAT below the panel's range, marginal USB sense, and copper under
the antenna. All are fixed and the board is rebuilt with 0 DRC violations.

Not ordered or tested on hardware. GUIDE.md lists what's still to check,
including J2's own PDF, the real cable fit and the battery behind the antenna.

Co-Authored-By: Claude Opus 5.5 <noreply@anthropic.com>
Claude-Session: https://claude.ai/code/session_01NGZp68ebE8nq2zT4H5x4dy
Parts:
- added C15: 1uF, Capacitor_SMD:C_0402_1005Metric, B.Cu at (111.3, 123.9)
- J2: value FH12-30S-0.5SH -> AFC07-S30ECC-00; footprint Connector_FFC-FPC:Hirose_FH12-30S-0.5SH_1x30-1MP_P0.50mm_Horizontal -> lumi:JUSHUO_AFC07-S30ECC-00
- R8: value 100k -> 150k
- moved C12 15.7 mm to (122.3, 123.9)
- moved C11 15.5 mm to (107.3, 123.9)
- moved R15 12.6 mm to (119.8, 123.9)
- moved C10 11.2 mm to (109.3, 123.9)
- moved C13 10.4 mm to (120.5, 121.1)
- moved R13 10.4 mm to (110.1, 121.1)
- moved C14 4.90 mm to (113.3, 123.9)
- moved R10 4.90 mm to (117.9, 123.9)
- moved TP1 1.00 mm to (101.4, 129.6)
- moved TP2 1.00 mm to (103.6, 129.6)
- moved J2 0.65 mm to (115.5, 128.6)
- moved TP3 0.55 mm to (101.4, 131.8)
- moved TP4 0.55 mm to (103.6, 131.8)
- moved TP5 0.40 mm to (125.6, 129.6)
- moved TP6 0.40 mm to (127.8, 129.6)
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Connections:
- J2 pad 11: 3V3 -> SDA
- J2 pad 12: GND -> SDA
- J2 pad 13: GND -> SCL
- J2 pad 14: OLED_RES -> GND
- J2 pad 17: GND -> OLED_RES
- J2 pad 18: SCL -> GND
- J2 pad 19: SDA -> GND
- J2 pad 2: C2P -> GND
- J2 pad 20: SDA -> 3V3
- J2 pad 22: GND -> 3V3
- J2 pad 24: GND -> (no net)
- J2 pad 25: GND -> VBAT
- J2 pad 26: IREF -> C1N
- J2 pad 27: VCOMH -> C1P
- J2 pad 28: VCC_OLED -> C2N
- J2 pad 29: GND -> C2P
- J2 pad 3: C2N -> VCC_OLED
- J2 pad 4: C1P -> VCOMH
- J2 pad 5: C1N -> IREF
- J2 pad 6: 3V3 -> GND
- J2 pad 7: (no net) -> GND
- J2 pad 9: 3V3 -> GND
Routing:
- net GND: track 178.1 -> 218.3 mm, vias 45 -> 30
- net IO8: track 10.9 -> 22.8 mm
- net USB_DP: track 18.5 -> 29.2 mm, vias 2 -> 3
- net IMU_INT: track 29.0 -> 18.3 mm, vias 2 -> 4
- net LDO_EN: track 38.2 -> 48.8 mm, vias 2 -> 4
- net VBAT: track 86.7 -> 80.0 mm
- net VBUS: track 31.2 -> 37.0 mm, vias 2 -> 3
- net PROG: track 3.29 -> 8.24 mm, vias 0 -> 2
- net VCC_OLED: track 7.56 -> 3.19 mm
- net EN: track 56.2 -> 59.2 mm, vias 2 -> 3
- net OLED_RES: track 11.7 -> 13.9 mm
- net SDA: track 32.5 -> 30.5 mm
- net USB_DN: track 23.9 -> 22.0 mm, vias 2 -> 0
- net C2P: track 2.23 -> 3.90 mm
- net SCL: track 27.5 -> 25.9 mm
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Other:
- outline, holes or cut-outs redrawn
- board text removed: "antenna: keep metal away"
