File: hardware/pcb/kicad/lumi/lumi.kicad_sch (KiCad schematic)
At the start: 44 parts, among them J1 USB-C 16P, J2 FH12-30S-0.5SH, SW1 MSK12C02, U1 ESP32-C3-WROOM-02-N4, U2 LIS2DH12TR, U3 TP4054, U4 RT9080-33GJ5

Commit message: Lumi PCB: rebuild in KiCad 10 with datasheet fixes
Checking the draft against the panel and Espressif datasheets found faults
the design-rule check can't see: a mirrored panel at J2, a bottom-contact
connector where the panel needs top contact, a screen cable that couldn't
reach, VBAT below the panel's range, marginal USB sense, and copper under
the antenna. All are fixed and the board is rebuilt with 0 DRC violations.

Not ordered or tested on hardware. GUIDE.md lists what's still to check,
including J2's own PDF, the real cable fit and the battery behind the antenna.

Co-Authored-By: Claude Opus 5.5 <noreply@anthropic.com>
Claude-Session: https://claude.ai/code/session_01NGZp68ebE8nq2zT4H5x4dy
Parts:
- added C15: 1uF, Capacitor_SMD:C_0402_1005Metric, symbol lumi:C15_1uF
- C14: Note Panel VDD/VBAT -> Panel VDD
- J2: value FH12-30S-0.5SH -> AFC07-S30ECC-00; footprint Connector_FFC-FPC:Hirose_FH12-30S-0.5SH_1x30-1MP_P0.50mm_Horizontal -> lumi:JUSHUO_AFC07-S30ECC-00; symbol lumi:J2_FH12-30S-0.5SH -> lumi:J2_AFC07-S30ECC-00; LCSC C506793 -> C11095; Note 30-pin 0.5 mm ZIF for the plug-in OLED. VERIFY contact side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 -> 30-pin 0.5 mm top-contact ZIF for the plug-in OLED (ER-OLED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
- R8: value 100k -> 150k; symbol lumi:R8_100k -> lumi:R8_150k; LCSC C25741 -> C25755; Note USB sense divider bottom -> USB sense divider bottom: 3.0 V from 5 V, clear of the C3's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
Connections:
- net 3V3: now also J2.20 (BS1), J2.22 (VDD); no longer J2.11 (BS1), J2.6 (VBAT), J2.9 (VDD)
- net C1N: now also J2.26 (C1N); no longer J2.5 (C1N)
- net C1P: now also J2.27 (C1P); no longer J2.4 (C1P)
- net C2N: now also J2.28 (C2N); no longer J2.3 (C2N)
- net C2P: now also J2.29 (C2P); no longer J2.2 (C2P)
- net GND: now also J1.SH (SHIELD), J2.14 (E/RD#), J2.18 (CS#), J2.19 (BS2), J2.2 (VLSS), J2.6 (D7), J2.7 (D6), J2.9 (D4), C15.2; no longer J1.S1 (SHIELD), J2.12 (BS2), J2.13 (CS#), J2.17 (E/RD#), J2.22 (D4), J2.24 (D6), J2.25 (D7), J2.29 (VLSS)
- net IREF: now also J2.5 (IREF); no longer J2.26 (IREF)
- net OLED_RES: now also J2.17 (RES#); no longer J2.14 (RES#)
- net SCL: now also J2.13 (D0/SCL); no longer J2.18 (D0/SCL)
- net SDA: now also J2.11 (D2/SDA), J2.12 (D1/SDA); no longer J2.19 (D1/SDA), J2.20 (D2/SDA)
- net VBAT: now also J2.25 (VBAT), C15.1
- net VCC_OLED: now also J2.3 (VCC); no longer J2.28 (VCC)
- net VCOMH: now also J2.4 (VCOMH); no longer J2.27 (VCOMH)
Other:
- note added: "OLED FPC, I2C 0x3C"
- note removed: "OLED FPC, I2C 0x3C (VERIFY pinout)"
- moved on the sheet: C9, R15, R5, R6, R7, R8
